File: hardware/mr_radar_ferret.sch (EAGLE design)
At the start: 91 parts

Commit message: component placement complete on ferret, layout partially complete. silkscreen cleanup and amplifier grounds remain
Parts:
- added C20: 100nF, pel_dipol_comp:CAPACITOR-0603
- added C45: 10uF, pel_dipol_comp:CAPACITOR-POLA
- added J$5, J$6: SMA_EDGE, SparkFun-Connectors:SMA_EDGE
- added JP3, JP4: (no value), SparkFun-Connectors:M03SCREW
- added R22, R23: 110, pel_dipol_comp:RESISTOR-0603
- added R8: 100, pel_dipol_comp:RESISTOR-0603
Connections:
- new net N$39: C9.1, J$5.SIGNAL, R5.1
- new net N$54: JP1.5, R11.2, U$12.VOUT@6
- net +10V: now also JP3.2, R22.2; no longer C31.1, C32.1, C33.1, C40.1, C41.1, C42.1, R1.2, R2.2
- net +5V: now also C20.1, C45.+, JP3.3, JP4.2, R23.2
- net GND: now also C20.2, C45.-, J$5.GND@0, J$5.GND@1, J$5.GND@2, J$5.GND@3, J$6.GND@0, J$6.GND@1, J$6.GND@2, J$6.GND@3, JP3.1, JP4.1, JP4.3, R8.2
- net N$1: now also R8.1
- net N$23: now also J$6.SIGNAL; no longer C9.1, R5.1
- net N$25: now also JP2.4; no longer JP2.1
- net N$42: now also JP2.3; no longer JP2.4
- net N$43: now also JP2.1, U$16.!CS@6; no longer R11.2, U$12.VOUT@6
- net N$44: now also JP2.2; no longer JP2.3
- net N$48: now also C31.1, C32.1, C33.1, C40.1, C41.1, C42.1, R1.2, R2.2, R22.1, R23.1; no longer JP2.2, U$16.!CS@6
- net VTUNE: no longer JP1.5
Other:
- moved on the sheet: C10, C18, C19, C21, C22, C23, C24, C25, C28, C29, C30, JP2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
