File: hardware/mr_radar_ferret.brd (EAGLE design)
At the start: 46.7 x 72.7 mm, 66 parts, among them U1 GALI-55+, U10 MAX2750, U11 GALI-55+, U12 AD5621, U13 REF2930, U3 GALI-55+, U4 GALI-55+, U7 DC25-73, U8 HMC213

Commit message: currently tested ferret r0, fixing a few bugs for the next revision, board layout of ferret now incomplete. isolation is much better than in platypus, but it is still a problem
Parts:
- R11: value JMP -> DNP
- moved U11 4.46 mm to (34.9, 57.8), turned to 270 degrees
- moved U4 4.46 mm to (34.9, 49.8), turned to 270 degrees
Connections:
- removed net N$19: C7.P$2, U11.RFIN
- removed net N$29: C17.P$2, U4.RFIN
- new net N$23: C7.P$2, U11.RFOUT
- new net N$9: C17.P$2, U4.RFOUT
- net N$18: now also U4.RFIN; no longer U4.RFOUT
- net N$20: now also U11.RFIN; no longer U11.RFOUT
Routing:
- net GND: track 66.5 -> 63.8 mm
- net N$29: track 2.30 -> 0.00 mm
- net N$19: track 1.66 -> 0.00 mm
- added copper zone on layer 1, net N$23
- added copper zone on layer 1, net N$9
- removed copper zone on layer 1, net N$19
- removed copper zone on layer 1, net N$29
Changed lines of the file:
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@@
 <attribute name="VALUE" x="33.9979" y="35.052" size="0.635" layer="27" font="vector" ratio="16" rot="R90"/>
 </element>
-<element name="U4" library="retro" package="SOT89" value="GALI-55+" x="30.48" y="50.165" smashed="yes" rot="R90">
-<attribute name="NAME" x="34.925" y="49.53" size="0.8128" layer="25" font="vector" ratio="16" rot="R90"/>
-<attribute name="VALUE" x="34.8249" y="47.7599" size="0.8128" layer="27" font="vector" ratio="16" rot="R90"/>
+<element name="U4" library="retro" package="SOT89" value="GALI-55+" x="34.925" y="49.8475" smashed="yes" rot="R270">
+<attribute name="NAME" x="30.48" y="50.4825" size="0.8128" layer="25" font="vector" ratio="16" rot="R270"/>
+<attribute name="VALUE" x="30.5801" y="52.2526" size="0.8128" layer="27" font="vector" ratio="16" rot="R270"/>
 </element>
 <element name="R3" library="pel_dipol_comp" package="0603-RES" value="110" x="28.2575" y="53.6575" smashed="yes" rot="R180">
@@
 <attribute name="VALUE" x="33.9979" y="53.1495" size="0.635" layer="27" font="vector" ratio="16" rot="R90"/>
 </element>
-<element name="U11" library="retro" package="SOT89" value="GALI-55+" x="30.48" y="58.1025" smashed="yes" rot="R90">
-<attribute name="NAME" x="34.925" y="56.8325" size="0.8128" layer="25" font="vector" ratio="16" rot="R90"/>
-<attribute name="VALUE" x="34.8249" y="55.6974" size="0.8128" layer="27" font="vector" ratio="16" rot="R90"/>
+<element name="U11" library="retro" package="SOT89" value="GALI-55+" x="34.925" y="57.785" smashed="yes" rot="R270">
+<attribute name="NAME" x="30.48" y="59.055" size="0.8128" layer="25" font="vector" ratio="16" rot="R270"/>
+<attribute name="VALUE" x="30.5801" y="60.1901" size="0.8128" layer="27" font="vector" ratio="16" rot="R270"/>
 </element>
 <element name="R4" library="pel_dipol_comp" package="0603-RES" value="110" x="28.2575" y="61.595" smashed="yes" rot="R180">
@@
 <attribute name="VALUE" x="10.9855" y="28.6004" size="0.635" layer="27" font="vector" ratio="16" rot="R180"/>
 </element>
-<element name="R11" library="pel_dipol_comp" package="0603-RES" value="JMP" x="5.715" y="17.78" smashed="yes" rot="R90">
+<element name="R11" library="pel_dipol_comp" package="0603-RES" value="DNP" x="5.715" y="17.78" smashed="yes" rot="R90">
 <attribute name="NAME" x="6.1468" y="19.4945" size="0.635" layer="25" font="vector" ratio="16" rot="R90"/>
 <attribute name="VALUE" x="7.0104" y="16.637" size="0.635" layer="27" font="vector" ratio="16" rot="R90"/>
@@
 <contactref element="U8" pad="8"/>
 <contactref element="U8" pad="6"/>
-<contactref element="U4" pad="GND"/>
-<contactref element="U4" pad="GNDPADDLE"/>
-<contactref element="U4" pad="GND"/>
-<contactref element="U4" pad="GNDPADDLE"/>
 <contactref element="U11" pad="GND"/>
 <contactref element="U11" pad="GNDPADDLE"/>
@@
 <via x="22.225" y="30.7975" extent="1-16" drill="0.5" shape="octagon"/>
 <wire x1="29.54" y1="32.385" x2="32.207" y2="32.385" width="0.4064" layer="1"/>
-<wire x1="29.54" y1="50.165" x2="32.207" y2="50.165" width="0.4064" layer="1"/>
-<wire x1="32.207" y1="58.1025" x2="29.54" y2="58.1025" width="0.4064" layer="1"/>
+<wire x1="33.198" y1="57.785" x2="35.865" y2="57.785" width="0.4064" layer="1"/>
 <wire x1="20.0025" y1="17.7675" x2="20.0025" y2="15.1005" width="0.4064" layer="1"/>
 <via x="26.035" y="58.7375" extent="1-16" drill="0.5" shape="octagon"/>
@@
 </polygon>
 <via x="35.2425" y="38.1" extent="1-16" drill="0.5" shape="octagon"/>
+<contactref element="U4" pad="GND"/>
+<contactref element="U4" pad="GND"/>
+<contactref element="U4" pad="GNDPADDLE"/>
+<contactref element="U4" pad="GNDPADDLE"/>
+<wire x1="30.7975" y1="58.1025" x2="33.198" y2="57.785" width="0" layer="19" extent="1-1"/>
+<wire x1="33.198" y1="49.8475" x2="30.7975" y2="50.165" width="0" layer="19" extent="1-1"/>
+<wire x1="35.865" y1="49.8475" x2="33.198" y2="49.8475" width="0" layer="19" extent="1-1"/>
 </signal>
 <signal name="N$2">
@@
 </signal>
 <signal name="N$18">
-<contactref element="U4" pad="RFOUT"/>
 <contactref element="C7" pad="P$1"/>
 <contactref element="L3" pad="P$2"/>
@@
 <wire x1="32.7025" y1="53.34" x2="32.7025" y2="52.07" width="1.524" layer="1"/>
 <wire x1="32.7025" y1="52.07" x2="32.7025" y2="51.9055" width="0.3048" layer="1"/>
-<wire x1="32.7025" y1="51.9055" x2="32.461" y2="51.664" width="0.3048" layer="1"/>
 <wire x1="31.5475" y1="53.6575" x2="32.5875" y2="53.6575" width="0.6096" layer="1"/>
 <wire x1="32.5875" y1="53.6575" x2="32.7025" y2="53.5425" width="0.6096" layer="1"/>
@@
 <vertex x="32.0675" y="53.975"/>
 </polygon>
+<contactref element="U4" pad="RFIN"/>
 </signal>
 <signal name="N$16">
@@
 </signal>
 <signal name="N$20">
-<contactref element="U11" pad="RFOUT"/>
 <contactref element="C8" pad="P$1"/>
 <contactref element="L4" pad="P$2"/>
@@
 <wire x1="32.7025" y1="61.2775" x2="32.7025" y2="60.0075" width="1.524" layer="1"/>
 <wire x1="32.7025" y1="60.0075" x2="32.461" y2="60.0075" width="0.3048" layer="1"/>
-<wire x1="32.461" y1="60.0075" x2="32.461" y2="59.6015" width="0.3048" layer="1"/>
 <wire x1="31.5475" y1="61.595" x2="32.7025" y2="61.595" width="0.6096" layer="1"/>
 <wire x1="32.7025" y1="61.595" x2="32.7025" y2="61.7975" width="0.6096" layer="1"/>
@@
 <vertex x="32.0675" y="61.9125"/>
 </polygon>
-</signal>
-<signal name="N$19">
 <contactref element="U11" pad="RFIN"/>
-<contactref element="C7" pad="P$2"/>
-<wire x1="32.461" y1="56.6035" x2="32.461" y2="56.439" width="0.3048" layer="1"/>
-<wire x1="32.461" y1="56.439" x2="32.7025" y2="56.1975" width="0.3048" layer="1"/>
-<wire x1="32.7025" y1="56.1975" x2="32.7025" y2="55.5625" width="1.524" layer="1"/>
-<wire x1="32.7025" y1="55.5625" x2="32.7025" y2="55.0425" width="0.3048" layer="1"/>
-<polygon width="0.254" layer="1" thermals="no">
-<vertex x="31.75" y="56.8325"/>
-<vertex x="33.3375" y="56.8325"/>
-<vertex x="33.655" y="56.515"/>
-<vertex x="33.655" y="55.245"/>
-<vertex x="33.3375" y="54.9275"/>
-<vertex x="32.0675" y="54.9275"/>
-<vertex x="31.75" y="55.245"/>
-</polygon>
 </signal>
 <signal name="N$22">
@@
 <wire x1="32.7025" y1="44.1325" x2="32.695" y2="44.125" width="0.4064" layer="1"/>
 <wire x1="32.695" y1="44.125" x2="32.695" y2="43.1325" width="0.4064" layer="1"/>
-</signal>
-<signal name="N$29">
-<contactref element="C17" pad="P$2"/>
-<contactref element="U4" pad="RFIN"/>
-<wire x1="32.461" y1="48.666" x2="32.7025" y2="48.4245" width="0.3048" layer="1"/>
-<wire x1="32.7025" y1="48.4245" x2="32.7025" y2="48.26" width="0.3048" layer="1"/>
-<wire x1="32.7025" y1="48.26" x2="32.7025" y2="47.3075" width="1.524" layer="1"/>
-<wire x1="32.7025" y1="47.3075" x2="32.7025" y2="46.47" width="0.3048" layer="1"/>
-<polygon width="0.254" layer="1" thermals="no">
-<vertex x="31.75" y="48.895"/>
-<vertex x="31.75" y="46.99"/>
-<vertex x="32.0675" y="46.6725"/>
-<vertex x="33.3375" y="46.6725"/>
-<vertex x="33.655" y="46.99"/>
-<vertex x="33.655" y="48.5775"/>
-<vertex x="33.3375" y="48.895"/>
-</polygon>
 </signal>
 <signal name="N$4">
@@
 <wire x1="19.8" y1="35.56" x2="20.32" y2="35.56" width="0.6096" layer="1"/>
 </signal>
+<signal name="N$9">
+<contactref element="U4" pad="RFOUT"/>
+<contactref element="C17" pad="P$2"/>
+<polygon width="0.254" layer="1" thermals="no">
+<vertex x="31.75" y="48.895"/>
+<vertex x="31.75" y="46.99"/>
+<vertex x="32.0675" y="46.6725"/>
+<vertex x="33.3375" y="46.6725"/>
+<vertex x="33.655" y="46.99"/>
+<vertex x="33.655" y="48.5775"/>
+<vertex x="33.3375" y="48.895"/>
+</polygon>
+</signal>
+<signal name="N$23">
+<contactref element="C7" pad="P$2"/>
+<contactref element="U11" pad="RFOUT"/>
+<polygon width="0.254" layer="1" thermals="no">
+<vertex x="31.75" y="56.8325"/>
+<vertex x="33.3375" y="56.8325"/>
+<vertex x="33.655" y="56.515"/>
+<vertex x="33.655" y="55.245"/>
+<vertex x="33.3375" y="54.9275"/>
+<vertex x="32.0675" y="54.9275"/>
+<vertex x="31.75" y="55.245"/>
+</polygon>
+</signal>
 </signals>
